File: hardware/gpio-only-hat/gpio-only-hat.kicad_sch (KiCad schematic)
At the start: 25 parts, among them J1 RPi_GPIO_40Pin, J2 GPIO4, J3 GPIO17, J4 GPIO18, J5 GPIO22, J6 GPIO23, J7 GPIO24, J8 GPIO25, J9 GPIO27

Commit message: rename: radxa → raspi (Raspberry Pi) im gesamten Projekt
Alle Referenzen auf "radxa" durch "raspi" bzw. "Raspberry Pi" ersetzt:
- Pfade: /etc/raspi_audio/, /opt/raspi_audio/
- Services: raspi-audio-web, raspi-audio-gpio
- Scripte: raspi_gpio.py, raspi_backup.zip
- Logs: raspi_install.log, raspi-network.log
- Kommentare und Dokumentation

Co-Authored-By: Claude Opus 4.6 <noreply@anthropic.com>
Other:
- note added: "Audio über 3.5mm Klinke des Raspberry Pi direkt"
- note removed: "Audio über 3.5mm Klinke des Pi/Radxa direkt"
Changed lines of the file:
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@@
   (text "RC-Entprellung: 10k + 100nF → τ ≈ 1ms" (at 120 230 0) (effects (font (size 1.5 1.5))))
   (text "Software-Debounce (200ms) kommt zusätzlich im GPIO-Daemon" (at 120 236 0) (effects (font (size 1.5 1.5))))
-  (text "Audio über 3.5mm Klinke des Pi/Radxa direkt" (at 120 242 0) (effects (font (size 1.5 1.5))))
+  (text "Audio über 3.5mm Klinke des Raspberry Pi direkt" (at 120 242 0) (effects (font (size 1.5 1.5))))
   (text "GPIO-Pins: 4, 17, 18, 22, 23, 24, 25, 27 (identisch mit app.py)" (at 120 248 0) (effects (font (size 1.5 1.5))))
 )
